Commit message: Fix xacro files
Fix xacro warnings #18

File: raspimouse_description/robots/raspimouse.urdf.xacro (robot description, xacro)
@@ -5,46 +5,40 @@
        xmlns:interface="http://playerstage.sourceforge.net/gazebo/xmlschema/#interface"
        xmlns:xacro="http://ros.org/wiki/xacro">
-  <xacro:include filename="$(find raspimouse_description)/urdf/body/body.urdf.xacro"/>
-  <xacro:include filename="$(find raspimouse_description)/urdf/wheel/wheel.urdf.xacro"/>
-  <xacro:include filename="$(find raspimouse_description)/urdf/sensors/lightsens.urdf.xacro"/>
+  <xacro:include filename="$(find raspimouse_description)/urdf/body/body.urdf.xacro" />
+  <xacro:include filename="$(find raspimouse_description)/urdf/wheel/wheel.urdf.xacro" />
+  <xacro:include filename="$(find raspimouse_description)/urdf/sensors/lightsens.urdf.xacro" />
   <!-- =============== Link & Joint =============== -->
   <!-- Base -->
-  <link name="base_footprint"/>
+  <link name="base_footprint" />
   <xacro:base parent="base_footprint">
-    <origin xyz="0 0 0.00185"/>
+    <origin xyz="0 0 0.00185" />
   </xacro:base>
   <!-- Wheel -->
   <xacro:wheel prefix="right" parent="base_link">
-    <origin xyz="0 -0.0425 0.02215" rpy="1.57 0 0"/>
-    <axis xyz="0 0 -1"/>
+    <origin xyz="0 -0.0425 0.02215" rpy="1.57 0 0" />
+    <axis xyz="0 0 -1" />
   </xacro:wheel>
   <xacro:wheel prefix="left" parent="base_link">
-    <origin xyz="0 0.0425 0.02215" rpy="-1.57 0 0"/>
-    <axis xyz="0 0 1"/>
+    <origin xyz="0 0.0425 0.02215" rpy="-1.57 0 0" />
+    <axis xyz="0 0 1" />
   </xacro:wheel>
   <!-- Sensors -->
   <xacro:light_sensor prefix="rf" parent="base_link">
-    <origin xyz="0.04 -0.045 0.032" rpy="0 0 0"/>
+    <origin xyz="0.04 -0.045 0.032" rpy="0 0 0" />
   </xacro:light_sensor>
   <xacro:light_sensor prefix="rs" parent="base_link">
-    <origin xyz="0.059 -0.01 0.032" rpy="0 0 -1.04"/>
+    <origin xyz="0.059 -0.01 0.032" rpy="0 0 -1.04" />
   </xacro:light_sensor>
   <xacro:light_sensor prefix="ls" parent="base_link">
-    <origin xyz="0.059 0.01 0.032" rpy="0 0 1.04"/>
+    <origin xyz="0.059 0.01 0.032" rpy="0 0 1.04" />
   </xacro:light_sensor>
   <xacro:light_sensor prefix="lf" parent="base_link">
-    <origin xyz="0.04 0.045 0.032" rpy="0 0 0"/>
+    <origin xyz="0.04 0.045 0.032" rpy="0 0 0" />
   </xacro:light_sensor>
   <!-- ===============  Transmission =============== -->
-  <!-- PositionJointInterface: requires position -->
-  <!-- <xacro:wheel_trans prefix="right" interface="PositionJointInterface"/> -->
-  <!-- <xacro:wheel_trans prefix="left" interface="PositionJointInterface"/>  -->
   <!-- VelocityJointInterface: requires position, velocity -->
   <!-- for DiffDriveController -->
-  <xacro:wheel_trans prefix="right" interface="hardware_interface/VelocityJointInterface"/>
-  <xacro:wheel_trans prefix="left" interface="hardware_interface/VelocityJointInterface"/>
-  <!-- EffortJointInterface: requires position, velocity, effort -->
-  <!-- <xacro:wheel_trans prefix="right" interface="EffortJointInterface"/> -->
-  <!-- <xacro:wheel_trans prefix="left" interface="EffortJointInterface"/>  -->
+  <xacro:wheel_trans prefix="right" interface="hardware_interface/VelocityJointInterface" />
+  <xacro:wheel_trans prefix="left" interface="hardware_interface/VelocityJointInterface" />
   <!-- =============== Gazebo =============== -->
   <gazebo>
@@ -56,11 +50,11 @@
   <xacro:base_gazebo/>
   <!-- Wheel -->
-  <xacro:wheel_gazebo prefix="right"/>
-  <xacro:wheel_gazebo prefix="left"/>
+  <xacro:wheel_gazebo prefix="right" />
+  <xacro:wheel_gazebo prefix="left" />
   <!-- Sensors -->
-  <xacro:lightsensor_gazebo prefix="rf" base_rad="0" rad_range="0.3" min_range="0.01" max_range="0.6"/>
-  <xacro:lightsensor_gazebo prefix="rs" base_rad="-1.04" rad_range="0.3" min_range="0.01" max_range="0.6"/>
-  <xacro:lightsensor_gazebo prefix="ls" base_rad="1.04" rad_range="0.3" min_range="0.01" max_range="0.6"/>
-  <xacro:lightsensor_gazebo prefix="lf" base_rad="0" rad_range="0.3" min_range="0.01" max_range="0.6"/>
+  <xacro:lightsensor_gazebo prefix="rf" base_rad="0" rad_range="0.3" min_range="0.01" max_range="0.6" />
+  <xacro:lightsensor_gazebo prefix="rs" base_rad="-1.04" rad_range="0.3" min_range="0.01" max_range="0.6" />
+  <xacro:lightsensor_gazebo prefix="ls" base_rad="1.04" rad_range="0.3" min_range="0.01" max_range="0.6" />
+  <xacro:lightsensor_gazebo prefix="lf" base_rad="0" rad_range="0.3" min_range="0.01" max_range="0.6" />
   <raspimouse_on_gazebo/>
 </robot>

File: raspimouse_description/robots/raspimouse_urg.urdf.xacro (robot description, xacro)
@@ -5,45 +5,44 @@
        xmlns:interface="http://playerstage.sourceforge.net/gazebo/xmlschema/#interface"
        xmlns:xacro="http://ros.org/wiki/xacro">
-  <xacro:include filename="$(find raspimouse_description)/urdf/body/body_urg.urdf.xacro"/>
-  <xacro:include filename="$(find raspimouse_description)/urdf/wheel/wheel.urdf.xacro"/>
-  <xacro:include filename="$(find raspimouse_description)/urdf/sensors/lightsens.urdf.xacro"/>
-  <xacro:include filename="$(find raspimouse_description)/urdf/sensors/lrf.urdf.xacro"/>
+  <xacro:include filename="$(find raspimouse_description)/urdf/body/body_urg.urdf.xacro" />
+  <xacro:include filename="$(find raspimouse_description)/urdf/wheel/wheel.urdf.xacro" />
+  <xacro:include filename="$(find raspimouse_description)/urdf/sensors/lightsens.urdf.xacro" />
+  <xacro:include filename="$(find raspimouse_description)/urdf/sensors/lrf.urdf.xacro" />
   <!-- =============== Link & Joint =============== -->
   <!-- Base -->
-  <link name="base_footprint"/>
+  <link name="base_footprint" />
   <xacro:base parent="base_footprint">
-    <origin xyz="0 0 0.00185"/>
+    <origin xyz="0 0 0.00185" />
   </xacro:base>
   <!-- Wheel -->
   <xacro:wheel prefix="right" parent="base_link">
-    <origin xyz="0 -0.0425 0.02215" rpy="1.57 0 0"/>
-    <axis xyz="0 0 -1"/>
+    <origin xyz="0 -0.0425 0.02215" rpy="1.57 0 0" />
+    <axis xyz="0 0 -1" />
   </xacro:wheel>
   <xacro:wheel prefix="left" parent="base_link">
-    <origin xyz="0 0.0425 0.02215" rpy="-1.57 0 0"/>
-    <axis xyz="0 0 1"/>
+    <origin xyz="0 0.0425 0.02215" rpy="-1.57 0 0" />
+    <axis xyz="0 0 1" />
   </xacro:wheel>
   <!-- Sensors -->
   <xacro:light_sensor prefix="rf" parent="base_link">
-    <origin xyz="0.04 -0.045 0.032" rpy="0 0 0"/>
+    <origin xyz="0.04 -0.045 0.032" rpy="0 0 0" />
   </xacro:light_sensor>
   <xacro:light_sensor prefix="rs" parent="base_link">
-    <origin xyz="0.059 -0.01 0.032" rpy="0 0 -1.04"/>
+    <origin xyz="0.059 -0.01 0.032" rpy="0 0 -1.04" />
   </xacro:light_sensor>
   <xacro:light_sensor prefix="ls" parent="base_link">
-    <origin xyz="0.059 0.01 0.032" rpy="0 0 1.04"/>
+    <origin xyz="0.059 0.01 0.032" rpy="0 0 1.04" />
   </xacro:light_sensor>
   <xacro:light_sensor prefix="lf" parent="base_link">
-    <origin xyz="0.04 0.045 0.032" rpy="0 0 0"/>
+    <origin xyz="0.04 0.045 0.032" rpy="0 0 0" />
   </xacro:light_sensor>
   <xacro:lrf_sensor prefix="urg_lrf_link" parent="base_link">
-    <origin xyz="0.0 0.0 0.14060" rpy="0 0 0"/>
-    <!-- <origin xyz="0.0 0.0 0.18745" rpy="0 0 0"/> -->
+    <origin xyz="0.0 0.0 0.14060" rpy="0 0 0" />
   </xacro:lrf_sensor>
   <!-- ===============  Transmission =============== -->
-  <!-- <xacro:wheel_trans prefix="right" interface="EffortJointInterface"/> -->
-  <!-- <xacro:wheel_trans prefix="left" interface="EffortJointInterface"/> -->
-  <xacro:wheel_trans prefix="right" interface="hardware_interface/VelocityJointInterface"/>
-  <xacro:wheel_trans prefix="left" interface="hardware_interface/VelocityJointInterface"/>
+  <!-- <xacro:wheel_trans prefix="right" interface="EffortJointInterface" /> -->
+  <!-- <xacro:wheel_trans prefix="left" interface="EffortJointInterface" /> -->
+  <xacro:wheel_trans prefix="right" interface="hardware_interface/VelocityJointInterface" />
+  <xacro:wheel_trans prefix="left" interface="hardware_interface/VelocityJointInterface" />
   <!-- =============== Gazebo =============== -->
   <gazebo>
@@ -55,12 +54,12 @@
   <xacro:base_gazebo/>
   <!-- Wheel -->
-  <xacro:wheel_gazebo prefix="right"/>
-  <xacro:wheel_gazebo prefix="left"/>
+  <xacro:wheel_gazebo prefix="right" />
+  <xacro:wheel_gazebo prefix="left" />
   <!-- Sensors -->
-  <xacro:lightsensor_gazebo prefix="rf" base_rad="0" rad_range="0.3" min_range="0.01" max_range="0.6"/>
-  <xacro:lightsensor_gazebo prefix="rs" base_rad="-1.04" rad_range="0.3" min_range="0.01" max_range="0.6"/>
-  <xacro:lightsensor_gazebo prefix="ls" base_rad="1.04" rad_range="0.3" min_range="0.01" max_range="0.6"/>
-  <xacro:lightsensor_gazebo prefix="lf" base_rad="0" rad_range="0.3" min_range="0.01" max_range="0.6"/>
-  <xacro:lrf_gazebo prefix="urg" base_rad="0" rad_range="4.71" min_range="0.10" max_range="5.6"/>
+  <xacro:lightsensor_gazebo prefix="rf" base_rad="0" rad_range="0.3" min_range="0.01" max_range="0.6" />
+  <xacro:lightsensor_gazebo prefix="rs" base_rad="-1.04" rad_range="0.3" min_range="0.01" max_range="0.6" />
+  <xacro:lightsensor_gazebo prefix="ls" base_rad="1.04" rad_range="0.3" min_range="0.01" max_range="0.6" />
+  <xacro:lightsensor_gazebo prefix="lf" base_rad="0" rad_range="0.3" min_range="0.01" max_range="0.6" />
+  <xacro:lrf_gazebo prefix="urg" base_rad="0" rad_range="4.71" min_range="0.10" max_range="5.6" />
   <raspimouse_on_gazebo/>
 </robot>

File: raspimouse_description/urdf/body/body.urdf.xacro (robot description, xacro)
@@ -1,22 +1,22 @@
 <?xml version="1.0"?>
 <robot xmlns:xacro="http://ros.org/wiki/xacro">
-  <xacro:include filename="$(find raspimouse_description)/urdf/body/body.gazebo.xacro"/>
+  <xacro:include filename="$(find raspimouse_description)/urdf/body/body.gazebo.xacro" />
   <xacro:property name="M_PI" value="3.1415926535897931" />
-  <xacro:property name="velocity_scale_factor" value="1.0"/>
+  <xacro:property name="velocity_scale_factor" value="1.0" />
   <xacro:macro name="base" params="parent *joint_origin">
     <joint name="base_joint" type="fixed">
-      <insert_block name="joint_origin"/>
-      <parent link="${parent}"/>
-      <child link="base_link"/>
+      <xacro:insert_block name="joint_origin" />
+      <parent link="${parent}" />
+      <child link="base_link" />
     </joint>
     <link name="base_link">
       <visual>
         <geometry>
-          <mesh filename="package://raspimouse_description/meshes/dae/body/RasPiMouse_body.dae"/>
+          <mesh filename="package://raspimouse_description/meshes/dae/body/RasPiMouse_body.dae" />
         </geometry>
       </visual>
       <collision>
         <geometry>
-          <mesh filename="package://raspimouse_description/meshes/dae/body/RasPiMouse_body.dae"/>
+          <mesh filename="package://raspimouse_description/meshes/dae/body/RasPiMouse_body.dae" />
         </geometry>
       </collision>
@@ -27,9 +27,9 @@
         <!-- NOTE END -->
         <!-- real origin -->
-        <!-- <origin xyz="&#45;0.005075 &#45;0.000427 0.029879"/> -->
+        <!-- <origin xyz="&#45;0.005075 &#45;0.000427 0.029879" /> -->
         <!-- virtual origin -->
-        <origin xyz="-0.001 0.0 0.029879"/>
-        <mass value="0.7186"/>
-        <inertia ixx="0.001238161833" ixy="0.000000904986" iyy="0.001368529369" ixz="0.000100297310" iyz="0.000022118177" izz="0.000784319117"/>
+        <origin xyz="-0.001 0.0 0.029879" />
+        <mass value="0.7186" />
+        <inertia ixx="0.001238161833" ixy="0.000000904986" iyy="0.001368529369" ixz="0.000100297310" iyz="0.000022118177" izz="0.000784319117" />
       </inertial>
     </link>

File: raspimouse_description/urdf/body/body_urg.urdf.xacro (robot description, xacro)
@@ -1,22 +1,22 @@
 <?xml version="1.0"?>
 <robot xmlns:xacro="http://ros.org/wiki/xacro">
-  <xacro:include filename="$(find raspimouse_description)/urdf/body/body_urg.gazebo.xacro"/>
+  <xacro:include filename="$(find raspimouse_description)/urdf/body/body_urg.gazebo.xacro" />
   <xacro:property name="M_PI" value="3.1415926535897931" />
-  <xacro:property name="velocity_scale_factor" value="1.0"/>
+  <xacro:property name="velocity_scale_factor" value="1.0" />
   <xacro:macro name="base" params="parent *joint_origin">
     <joint name="base_joint" type="fixed">
-      <insert_block name="joint_origin"/>
-      <parent link="${parent}"/>
-      <child link="base_link"/>
+      <xacro:insert_block name="joint_origin" />
+      <parent link="${parent}" />
+      <child link="base_link" />
     </joint>
     <link name="base_link">
       <visual>
         <geometry>
-          <mesh filename="package://raspimouse_description/meshes/dae/body/RasPiMouse_body-TopPlate.dae"/>
+          <mesh filename="package://raspimouse_description/meshes/dae/body/RasPiMouse_body-TopPlate.dae" />
         </geometry>
       </visual>
       <collision>
         <geometry>
-          <mesh filename="package://raspimouse_description/meshes/dae/body/RasPiMouse_body-TopPlate.dae"/>
+          <mesh filename="package://raspimouse_description/meshes/dae/body/RasPiMouse_body-TopPlate.dae" />
         </geometry>
       </collision>
@@ -27,9 +27,9 @@
         <!-- NOTE END -->
         <!-- real origin -->
-        <!-- <origin xyz="&#45;0.003851 &#45;0.000443 0.031714"/> -->
+        <!-- <origin xyz="&#45;0.003851 &#45;0.000443 0.031714" /> -->
         <!-- virtual origin -->
-        <origin xyz="-0.000851 -0.000003 0.031714"/>
-        <mass value="0.759881"/>
-        <inertia ixx="0.001561279589" ixy="0.00000150035" iyy="0.001698462955" ixz="0.000042679786" iyz="0.000023629024" izz="0.000855782529"/>
+        <origin xyz="-0.000851 -0.000003 0.031714" />
+        <mass value="0.759881" />
+        <inertia ixx="0.001561279589" ixy="0.00000150035" iyy="0.001698462955" ixz="0.000042679786" iyz="0.000023629024" izz="0.000855782529" />
       </inertial>
     </link>

File: raspimouse_description/urdf/raspimouse.urdf.xacro (robot description, xacro)
@@ -1,66 +1 @@
-<?xml version="1.0"?>
-<robot name="raspimouse_on_gazebo"
-       xmlns:sensor="http://playerstage.sourceforge.net/gazebo/xmlschema/#sensor"
-       xmlns:controller="http://playerstage.sourceforge.net/gazebo/xmlschema/#controller"
-       xmlns:interface="http://playerstage.sourceforge.net/gazebo/xmlschema/#interface"
-       xmlns:xacro="http://ros.org/wiki/xacro">
-  <xacro:include filename="$(find raspimouse_description)/urdf/body/body.urdf.xacro"/>
-  <xacro:include filename="$(find raspimouse_description)/urdf/wheel/wheel.urdf.xacro"/>
-  <xacro:include filename="$(find raspimouse_description)/urdf/sensors/lightsens.urdf.xacro"/>
-  <!-- =============== Link & Joint =============== -->
-  <!-- Base -->
-  <link name="base_footprint"/>
-  <xacro:base parent="base_footprint">
-    <origin xyz="0 0 0.00185"/>
-  </xacro:base>
-  <!-- Wheel -->
-  <xacro:wheel prefix="right" parent="base_link">
-    <origin xyz="0 -0.0425 0.02215" rpy="1.57 0 0"/>
-    <axis xyz="0 0 -1"/>
-  </xacro:wheel>
-  <xacro:wheel prefix="left" parent="base_link">
-    <origin xyz="0 0.0425 0.02215" rpy="-1.57 0 0"/>
-    <axis xyz="0 0 1"/>
-  </xacro:wheel>
-  <!-- Sensors -->
-  <xacro:light_sensor prefix="rf" parent="base_link">
-    <origin xyz="0.04 -0.045 0.032" rpy="0 0 0"/>
-  </xacro:light_sensor>
-  <xacro:light_sensor prefix="rs" parent="base_link">
-    <origin xyz="0.059 -0.01 0.032" rpy="0 0 -1.04"/>
-  </xacro:light_sensor>
-  <xacro:light_sensor prefix="ls" parent="base_link">
-    <origin xyz="0.059 0.01 0.032" rpy="0 0 1.04"/>
-  </xacro:light_sensor>
-  <xacro:light_sensor prefix="lf" parent="base_link">
-    <origin xyz="0.04 0.045 0.032" rpy="0 0 0"/>
-  </xacro:light_sensor>
-  <!-- ===============  Transmission =============== -->
-  <!-- PositionJointInterface: requires position -->
-  <!-- <xacro:wheel_trans prefix="right" interface="PositionJointInterface"/> -->
-  <!-- <xacro:wheel_trans prefix="left" interface="PositionJointInterface"/>  -->
-  <!-- VelocityJointInterface: requires position, velocity -->
-  <!-- for DiffDriveController -->
-  <xacro:wheel_trans prefix="right" interface="hardware_interface/VelocityJointInterface"/>
-  <xacro:wheel_trans prefix="left" interface="hardware_interface/VelocityJointInterface"/>
-  <!-- EffortJointInterface: requires position, velocity, effort -->
-  <!-- <xacro:wheel_trans prefix="right" interface="EffortJointInterface"/> -->
-  <!-- <xacro:wheel_trans prefix="left" interface="EffortJointInterface"/>  -->
-  <!-- =============== Gazebo =============== -->
-  <gazebo>
-    <plugin name="gazebo_ros_control" filename="libgazebo_ros_control.so">
-      <robotNamespace>raspimouse_on_gazebo</robotNamespace>
-    </plugin>
-  </gazebo>
-  <!-- Base -->
-  <xacro:base_gazebo/>
-  <!-- Wheel -->
-  <xacro:wheel_gazebo prefix="right"/>
-  <xacro:wheel_gazebo prefix="left"/>
-  <!-- Sensors -->
-  <xacro:lightsensor_gazebo prefix="rf" base_rad="0" rad_range="0.3" min_range="0.01" max_range="0.6"/>
-  <xacro:lightsensor_gazebo prefix="rs" base_rad="-1.04" rad_range="0.3" min_range="0.01" max_range="0.6"/>
-  <xacro:lightsensor_gazebo prefix="ls" base_rad="1.04" rad_range="0.3" min_range="0.01" max_range="0.6"/>
-  <xacro:lightsensor_gazebo prefix="lf" base_rad="0" rad_range="0.3" min_range="0.01" max_range="0.6"/>
-  <raspimouse_on_gazebo/>
-</robot>
+../robots/raspimouse.urdf.xacro

File: raspimouse_description/urdf/raspimouse_urg.urdf.xacro (robot description, xacro)
@@ -1,66 +1 @@
-<?xml version="1.0"?>
-<robot name="raspimouse_on_gazebo"
-       xmlns:sensor="http://playerstage.sourceforge.net/gazebo/xmlschema/#sensor"
-       xmlns:controller="http://playerstage.sourceforge.net/gazebo/xmlschema/#controller"
-       xmlns:interface="http://playerstage.sourceforge.net/gazebo/xmlschema/#interface"
-       xmlns:xacro="http://ros.org/wiki/xacro">
-  <xacro:include filename="$(find raspimouse_description)/urdf/body/body_urg.urdf.xacro"/>
-  <xacro:include filename="$(find raspimouse_description)/urdf/wheel/wheel.urdf.xacro"/>
-  <xacro:include filename="$(find raspimouse_description)/urdf/sensors/lightsens.urdf.xacro"/>
-  <xacro:include filename="$(find raspimouse_description)/urdf/sensors/lrf.urdf.xacro"/>
-  <!-- =============== Link & Joint =============== -->
-  <!-- Base -->
-  <link name="base_footprint"/>
-  <xacro:base parent="base_footprint">
-    <origin xyz="0 0 0.00185"/>
-  </xacro:base>
-  <!-- Wheel -->
-  <xacro:wheel prefix="right" parent="base_link">
-    <origin xyz="0 -0.0425 0.02215" rpy="1.57 0 0"/>
-    <axis xyz="0 0 -1"/>
-  </xacro:wheel>
-  <xacro:wheel prefix="left" parent="base_link">
-    <origin xyz="0 0.0425 0.02215" rpy="-1.57 0 0"/>
-    <axis xyz="0 0 1"/>
-  </xacro:wheel>
-  <!-- Sensors -->
-  <xacro:light_sensor prefix="rf" parent="base_link">
-    <origin xyz="0.04 -0.045 0.032" rpy="0 0 0"/>
-  </xacro:light_sensor>
-  <xacro:light_sensor prefix="rs" parent="base_link">
-    <origin xyz="0.059 -0.01 0.032" rpy="0 0 -1.04"/>
-  </xacro:light_sensor>
-  <xacro:light_sensor prefix="ls" parent="base_link">
-    <origin xyz="0.059 0.01 0.032" rpy="0 0 1.04"/>
-  </xacro:light_sensor>
-  <xacro:light_sensor prefix="lf" parent="base_link">
-    <origin xyz="0.04 0.045 0.032" rpy="0 0 0"/>
-  </xacro:light_sensor>
-  <xacro:lrf_sensor prefix="urg_lrf_link" parent="base_link">
-    <origin xyz="0.0 0.0 0.14060" rpy="0 0 0"/>
-    <!-- <origin xyz="0.0 0.0 0.18745" rpy="0 0 0"/> -->
-  </xacro:lrf_sensor>
-  <!-- ===============  Transmission =============== -->
-  <!-- <xacro:wheel_trans prefix="right" interface="EffortJointInterface"/> -->
-  <!-- <xacro:wheel_trans prefix="left" interface="EffortJointInterface"/> -->
-  <xacro:wheel_trans prefix="right" interface="hardware_interface/VelocityJointInterface"/>
-  <xacro:wheel_trans prefix="left" interface="hardware_interface/VelocityJointInterface"/>
-  <!-- =============== Gazebo =============== -->
-  <gazebo>
-    <plugin name="gazebo_ros_control" filename="libgazebo_ros_control.so">
-      <robotNamespace>raspimouse_on_gazebo</robotNamespace>
-    </plugin>
-  </gazebo>
-  <!-- Base -->
-  <xacro:base_gazebo/>
-  <!-- Wheel -->
-  <xacro:wheel_gazebo prefix="right"/>
-  <xacro:wheel_gazebo prefix="left"/>
-  <!-- Sensors -->
-  <xacro:lightsensor_gazebo prefix="rf" base_rad="0" rad_range="0.3" min_range="0.01" max_range="0.6"/>
-  <xacro:lightsensor_gazebo prefix="rs" base_rad="-1.04" rad_range="0.3" min_range="0.01" max_range="0.6"/>
-  <xacro:lightsensor_gazebo prefix="ls" base_rad="1.04" rad_range="0.3" min_range="0.01" max_range="0.6"/>
-  <xacro:lightsensor_gazebo prefix="lf" base_rad="0" rad_range="0.3" min_range="0.01" max_range="0.6"/>
-  <xacro:lrf_gazebo prefix="urg" base_rad="0" rad_range="4.71" min_range="0.10" max_range="5.6"/>
-  <raspimouse_on_gazebo/>
-</robot>
+../robots/raspimouse_urg.urdf.xacro

File: raspimouse_description/urdf/sensors/lightsens.urdf.xacro (robot description, xacro)
@@ -1,10 +1,10 @@
 <?xml version="1.0"?>
 <robot name="light_sensor" xmlns:xacro="http://ros.org/wiki/xacro">
-  <xacro:include filename="$(find raspimouse_description)/urdf/sensors/lightsens.gazebo.xacro"/>
+  <xacro:include filename="$(find raspimouse_description)/urdf/sensors/lightsens.gazebo.xacro" />
   <xacro:macro name="light_sensor" params="prefix parent *joint_origin">
     <joint name="${prefix}_joint" type="fixed">
-      <insert_block name="joint_origin"/>
-      <parent link="${parent}"/>
-      <child link="${prefix}"/>
+      <xacro:insert_block name="joint_origin" />
+      <parent link="${parent}" />
+      <child link="${prefix}" />
     </joint>
     <link name="${prefix}">
@@ -15,5 +15,5 @@
       </visual>
       <material name="grey">
-        <color rgba="0.5 0.5 0.5 1"/>
+        <color rgba="0.5 0.5 0.5 1" />
       </material>
       <inertial>

File: raspimouse_description/urdf/sensors/lrf.urdf.xacro (robot description, xacro)
@@ -1,20 +1,20 @@
 <?xml version="1.0"?>
 <robot name="light_sensor" xmlns:xacro="http://ros.org/wiki/xacro">
-  <xacro:include filename="$(find raspimouse_description)/urdf/sensors/lrf.gazebo.xacro"/>
+  <xacro:include filename="$(find raspimouse_description)/urdf/sensors/lrf.gazebo.xacro" />
   <xacro:macro name="lrf_sensor" params="prefix parent *joint_origin">
     <joint name="${prefix}_joint" type="fixed">
-      <insert_block name="joint_origin"/>
-      <parent link="${parent}"/>
-      <child link="${prefix}"/>
+      <xacro:insert_block name="joint_origin" />
+      <parent link="${parent}" />
+      <child link="${prefix}" />
     </joint>
     <link name="${prefix}">
       <visual>
         <geometry>
-          <mesh filename="package://raspimouse_description/meshes/dae/sensor/URG_center.dae"/>
+          <mesh filename="package://raspimouse_description/meshes/dae/sensor/URG_center.dae" />
         </geometry>
       </visual>
       <collision>
         <geometry>
-          <mesh filename="package://raspimouse_description/meshes/dae/sensor/URG_center.dae"/>
+          <mesh filename="package://raspimouse_description/meshes/dae/sensor/URG_center.dae" />
         </geometry>
       </collision>
