Commit message: Fix xacro files
Fix xacro warnings #18

File: raspimouse_description/urdf/wheel/wheel.urdf.xacro (robot description, xacro)
@@ -1,17 +1,16 @@
 <?xml version="1.0"?>
 <robot xmlns:xacro="http://ros.org/wiki/xacro">
-  <xacro:include filename="$(find raspimouse_description)/urdf/wheel/wheel.transmission.xacro"/>
-  <xacro:include filename="$(find raspimouse_description)/urdf/wheel/wheel.gazebo.xacro"/>
-  <!-- <property name="wheel_radius" value="0.0239"/> -->
-  <property name="wheel_radius" value="0.0249"/>
-  <property name="wheel_length" value="0.01"/>
-  <property name="wheel_mass" value="0.0113"/>
+  <xacro:include filename="$(find raspimouse_description)/urdf/wheel/wheel.transmission.xacro" />
+  <xacro:include filename="$(find raspimouse_description)/urdf/wheel/wheel.gazebo.xacro" />
+  <xacro:property name="wheel_radius" value="0.024" />
+  <xacro:property name="wheel_length" value="0.01" />
+  <xacro:property name="wheel_mass" value="0.0113" />
   <xacro:macro name="wheel" params="prefix parent *joint_origin *joint_axis">
   <joint name="${prefix}_wheel_joint" type="continuous">
-    <insert_block name="joint_origin"/>
-    <insert_block name="joint_axis"/>
-    <parent link="${parent}"/>
-    <child link="${prefix}_wheel"/>
-    <limit effort="70" velocity="15"/>
+    <xacro:insert_block name="joint_origin" />
+    <xacro:insert_block name="joint_axis" />
+    <parent link="${parent}" />
+    <child link="${prefix}_wheel" />
+    <limit effort="70" velocity="15" />
     <safety_controller  k_velocity="10" />
     <dynamics damping="1.0" friction="1.0" />
@@ -20,18 +19,17 @@
     <visual>
       <geometry>
-        <mesh filename="package://raspimouse_description/meshes/dae/wheel/RasPiMouse_wheel.dae"/>
+        <mesh filename="package://raspimouse_description/meshes/dae/wheel/RasPiMouse_wheel.dae" />
       </geometry>
     </visual>
     <collision>
-      <!-- <insert_block name="joint_origin"/> -->
         <geometry>
-          <!-- <cylinder radius="${wheel_radius}" length="${wheel_length}"/> -->
-          <mesh filename="package://raspimouse_description/meshes/dae/wheel/RasPiMouse_wheel.dae"/>
+          <!-- <cylinder radius="${wheel_radius}" length="${wheel_length}" /> -->
+          <mesh filename="package://raspimouse_description/meshes/dae/wheel/RasPiMouse_wheel.dae" />
         </geometry>
     </collision>
       <inertial>
-        <origin xyz="-0.000107 0 0.002875"/>
-        <mass value="${wheel_mass}"/>
-        <inertia ixx="0.000002208187" ixy="0.000000000001" iyy="0.00000218412" ixz="0.000000004787" iyz="0.000000000003" izz="0.000004078299"/>
+        <origin xyz="-0.000107 0 0.002875" />
+        <mass value="${wheel_mass}" />
+        <inertia ixx="0.000002208187" ixy="0.000000000001" iyy="0.00000218412" ixz="0.000000004787" iyz="0.000000000003" izz="0.000004078299" />
       </inertial>
   </link>

File: raspimouse_gazebo/materials/sample_maze.wall.xacro (robot description, xacro)
@@ -4,5 +4,5 @@
     <model name='wall'>
       <!-- <pose>&#45;0.09 0 0.5 0 0 1.57</pose> -->
-      <insert_block name="pose"/>
+      <xacro:insert_block name="pose" />
       <link name='link'>
         <inertial>

File: raspimouse_gazebo/materials/sample_maze.world.xacro (robot description, xacro)
@@ -2,9 +2,9 @@
 <sdf version="1.4" xmlns:xacro="http://ros.org/wiki/xacro">
 <!-- <sdf version="1.4"> -->
-<xacro:include filename="$(find raspimouse_gazebo)/materials/sample_maze.wall.xacro"/>
+<xacro:include filename="$(find raspimouse_gazebo)/materials/sample_maze.wall.xacro" />
 <world name="default">
-  <include>
+  <xacro:include>
     <uri>model://ground_plane</uri>
-  </include>
+  </xacro:include>
   <light name='sun' type='directional'>
     <cast_shadows>1</cast_shadows>

Commit message: Fix xacro files
Fix xacro warnings #18

Conflicts:
	raspimouse_description/urdf/raspimouse.urdf.xacro
	raspimouse_description/urdf/raspimouse_urg.urdf.xacro

File: raspimouse_description/robots/raspimouse.urdf.xacro (robot description, xacro)
@@ -5,46 +5,40 @@
        xmlns:interface="http://playerstage.sourceforge.net/gazebo/xmlschema/#interface"
        xmlns:xacro="http://ros.org/wiki/xacro">
-  <xacro:include filename="$(find raspimouse_description)/urdf/body/body.urdf.xacro"/>
-  <xacro:include filename="$(find raspimouse_description)/urdf/wheel/wheel.urdf.xacro"/>
-  <xacro:include filename="$(find raspimouse_description)/urdf/sensors/lightsens.urdf.xacro"/>
+  <xacro:include filename="$(find raspimouse_description)/urdf/body/body.urdf.xacro" />
+  <xacro:include filename="$(find raspimouse_description)/urdf/wheel/wheel.urdf.xacro" />
+  <xacro:include filename="$(find raspimouse_description)/urdf/sensors/lightsens.urdf.xacro" />
   <!-- =============== Link & Joint =============== -->
   <!-- Base -->
-  <link name="base_footprint"/>
+  <link name="base_footprint" />
   <xacro:base parent="base_footprint">
-    <origin xyz="0 0 0.00185"/>
+    <origin xyz="0 0 0.00185" />
   </xacro:base>
   <!-- Wheel -->
   <xacro:wheel prefix="right" parent="base_link">
-    <origin xyz="0 -0.0425 0.02215" rpy="1.57 0 0"/>
-    <axis xyz="0 0 -1"/>
+    <origin xyz="0 -0.0425 0.02215" rpy="1.57 0 0" />
+    <axis xyz="0 0 -1" />
   </xacro:wheel>
   <xacro:wheel prefix="left" parent="base_link">
-    <origin xyz="0 0.0425 0.02215" rpy="-1.57 0 0"/>
-    <axis xyz="0 0 1"/>
+    <origin xyz="0 0.0425 0.02215" rpy="-1.57 0 0" />
+    <axis xyz="0 0 1" />
   </xacro:wheel>
   <!-- Sensors -->
   <xacro:light_sensor prefix="rf" parent="base_link">
-    <origin xyz="0.04 -0.045 0.032" rpy="0 0 0"/>
+    <origin xyz="0.04 -0.045 0.032" rpy="0 0 0" />
   </xacro:light_sensor>
   <xacro:light_sensor prefix="rs" parent="base_link">
-    <origin xyz="0.059 -0.01 0.032" rpy="0 0 -1.04"/>
+    <origin xyz="0.059 -0.01 0.032" rpy="0 0 -1.04" />
   </xacro:light_sensor>
   <xacro:light_sensor prefix="ls" parent="base_link">
-    <origin xyz="0.059 0.01 0.032" rpy="0 0 1.04"/>
+    <origin xyz="0.059 0.01 0.032" rpy="0 0 1.04" />
   </xacro:light_sensor>
   <xacro:light_sensor prefix="lf" parent="base_link">
-    <origin xyz="0.04 0.045 0.032" rpy="0 0 0"/>
+    <origin xyz="0.04 0.045 0.032" rpy="0 0 0" />
   </xacro:light_sensor>
   <!-- ===============  Transmission =============== -->
-  <!-- PositionJointInterface: requires position -->
-  <!-- <xacro:wheel_trans prefix="right" interface="PositionJointInterface"/> -->
-  <!-- <xacro:wheel_trans prefix="left" interface="PositionJointInterface"/>  -->
   <!-- VelocityJointInterface: requires position, velocity -->
   <!-- for DiffDriveController -->
-  <xacro:wheel_trans prefix="right" interface="hardware_interface/VelocityJointInterface"/>
-  <xacro:wheel_trans prefix="left" interface="hardware_interface/VelocityJointInterface"/>
-  <!-- EffortJointInterface: requires position, velocity, effort -->
-  <!-- <xacro:wheel_trans prefix="right" interface="EffortJointInterface"/> -->
-  <!-- <xacro:wheel_trans prefix="left" interface="EffortJointInterface"/>  -->
+  <xacro:wheel_trans prefix="right" interface="VelocityJointInterface" />
+  <xacro:wheel_trans prefix="left" interface="VelocityJointInterface" />
   <!-- =============== Gazebo =============== -->
   <gazebo>
@@ -56,11 +50,11 @@
   <xacro:base_gazebo/>
   <!-- Wheel -->
-  <xacro:wheel_gazebo prefix="right"/>
-  <xacro:wheel_gazebo prefix="left"/>
+  <xacro:wheel_gazebo prefix="right" />
+  <xacro:wheel_gazebo prefix="left" />
   <!-- Sensors -->
-  <xacro:lightsensor_gazebo prefix="rf" base_rad="0" rad_range="0.3" min_range="0.01" max_range="0.6"/>
-  <xacro:lightsensor_gazebo prefix="rs" base_rad="-1.04" rad_range="0.3" min_range="0.01" max_range="0.6"/>
-  <xacro:lightsensor_gazebo prefix="ls" base_rad="1.04" rad_range="0.3" min_range="0.01" max_range="0.6"/>
-  <xacro:lightsensor_gazebo prefix="lf" base_rad="0" rad_range="0.3" min_range="0.01" max_range="0.6"/>
+  <xacro:lightsensor_gazebo prefix="rf" base_rad="0" rad_range="0.3" min_range="0.01" max_range="0.6" />
+  <xacro:lightsensor_gazebo prefix="rs" base_rad="-1.04" rad_range="0.3" min_range="0.01" max_range="0.6" />
+  <xacro:lightsensor_gazebo prefix="ls" base_rad="1.04" rad_range="0.3" min_range="0.01" max_range="0.6" />
+  <xacro:lightsensor_gazebo prefix="lf" base_rad="0" rad_range="0.3" min_range="0.01" max_range="0.6" />
   <raspimouse_on_gazebo/>
 </robot>

File: raspimouse_description/robots/raspimouse_urg.urdf.xacro (robot description, xacro)
@@ -5,45 +5,44 @@
        xmlns:interface="http://playerstage.sourceforge.net/gazebo/xmlschema/#interface"
        xmlns:xacro="http://ros.org/wiki/xacro">
-  <xacro:include filename="$(find raspimouse_description)/urdf/body/body_urg.urdf.xacro"/>
-  <xacro:include filename="$(find raspimouse_description)/urdf/wheel/wheel.urdf.xacro"/>
-  <xacro:include filename="$(find raspimouse_description)/urdf/sensors/lightsens.urdf.xacro"/>
-  <xacro:include filename="$(find raspimouse_description)/urdf/sensors/lrf.urdf.xacro"/>
+  <xacro:include filename="$(find raspimouse_description)/urdf/body/body_urg.urdf.xacro" />
+  <xacro:include filename="$(find raspimouse_description)/urdf/wheel/wheel.urdf.xacro" />
+  <xacro:include filename="$(find raspimouse_description)/urdf/sensors/lightsens.urdf.xacro" />
+  <xacro:include filename="$(find raspimouse_description)/urdf/sensors/lrf.urdf.xacro" />
   <!-- =============== Link & Joint =============== -->
   <!-- Base -->
-  <link name="base_footprint"/>
+  <link name="base_footprint" />
   <xacro:base parent="base_footprint">
-    <origin xyz="0 0 0.00185"/>
+    <origin xyz="0 0 0.00185" />
   </xacro:base>
   <!-- Wheel -->
   <xacro:wheel prefix="right" parent="base_link">
-    <origin xyz="0 -0.0425 0.02215" rpy="1.57 0 0"/>
-    <axis xyz="0 0 -1"/>
+    <origin xyz="0 -0.0425 0.02215" rpy="1.57 0 0" />
+    <axis xyz="0 0 -1" />
   </xacro:wheel>
   <xacro:wheel prefix="left" parent="base_link">
-    <origin xyz="0 0.0425 0.02215" rpy="-1.57 0 0"/>
-    <axis xyz="0 0 1"/>
+    <origin xyz="0 0.0425 0.02215" rpy="-1.57 0 0" />
+    <axis xyz="0 0 1" />
   </xacro:wheel>
   <!-- Sensors -->
   <xacro:light_sensor prefix="rf" parent="base_link">
-    <origin xyz="0.04 -0.045 0.032" rpy="0 0 0"/>
+    <origin xyz="0.04 -0.045 0.032" rpy="0 0 0" />
   </xacro:light_sensor>
   <xacro:light_sensor prefix="rs" parent="base_link">
-    <origin xyz="0.059 -0.01 0.032" rpy="0 0 -1.04"/>
+    <origin xyz="0.059 -0.01 0.032" rpy="0 0 -1.04" />
   </xacro:light_sensor>
   <xacro:light_sensor prefix="ls" parent="base_link">
-    <origin xyz="0.059 0.01 0.032" rpy="0 0 1.04"/>
+    <origin xyz="0.059 0.01 0.032" rpy="0 0 1.04" />
   </xacro:light_sensor>
   <xacro:light_sensor prefix="lf" parent="base_link">
-    <origin xyz="0.04 0.045 0.032" rpy="0 0 0"/>
+    <origin xyz="0.04 0.045 0.032" rpy="0 0 0" />
   </xacro:light_sensor>
   <xacro:lrf_sensor prefix="urg_lrf_link" parent="base_link">
-    <origin xyz="0.0 0.0 0.14060" rpy="0 0 0"/>
-    <!-- <origin xyz="0.0 0.0 0.18745" rpy="0 0 0"/> -->
+    <origin xyz="0.0 0.0 0.14060" rpy="0 0 0" />
   </xacro:lrf_sensor>
   <!-- ===============  Transmission =============== -->
-  <!-- <xacro:wheel_trans prefix="right" interface="EffortJointInterface"/> -->
-  <!-- <xacro:wheel_trans prefix="left" interface="EffortJointInterface"/> -->
-  <xacro:wheel_trans prefix="right" interface="hardware_interface/VelocityJointInterface"/>
-  <xacro:wheel_trans prefix="left" interface="hardware_interface/VelocityJointInterface"/>
+  <!-- <xacro:wheel_trans prefix="right" interface="EffortJointInterface" /> -->
+  <!-- <xacro:wheel_trans prefix="left" interface="EffortJointInterface" /> -->
+  <xacro:wheel_trans prefix="right" interface="VelocityJointInterface" />
+  <xacro:wheel_trans prefix="left" interface="VelocityJointInterface" />
   <!-- =============== Gazebo =============== -->
   <gazebo>
@@ -55,12 +54,12 @@
   <xacro:base_gazebo/>
   <!-- Wheel -->
-  <xacro:wheel_gazebo prefix="right"/>
-  <xacro:wheel_gazebo prefix="left"/>
+  <xacro:wheel_gazebo prefix="right" />
+  <xacro:wheel_gazebo prefix="left" />
   <!-- Sensors -->
-  <xacro:lightsensor_gazebo prefix="rf" base_rad="0" rad_range="0.3" min_range="0.01" max_range="0.6"/>
-  <xacro:lightsensor_gazebo prefix="rs" base_rad="-1.04" rad_range="0.3" min_range="0.01" max_range="0.6"/>
-  <xacro:lightsensor_gazebo prefix="ls" base_rad="1.04" rad_range="0.3" min_range="0.01" max_range="0.6"/>
-  <xacro:lightsensor_gazebo prefix="lf" base_rad="0" rad_range="0.3" min_range="0.01" max_range="0.6"/>
-  <xacro:lrf_gazebo prefix="urg" base_rad="0" rad_range="4.71" min_range="0.10" max_range="5.6"/>
+  <xacro:lightsensor_gazebo prefix="rf" base_rad="0" rad_range="0.3" min_range="0.01" max_range="0.6" />
+  <xacro:lightsensor_gazebo prefix="rs" base_rad="-1.04" rad_range="0.3" min_range="0.01" max_range="0.6" />
+  <xacro:lightsensor_gazebo prefix="ls" base_rad="1.04" rad_range="0.3" min_range="0.01" max_range="0.6" />
+  <xacro:lightsensor_gazebo prefix="lf" base_rad="0" rad_range="0.3" min_range="0.01" max_range="0.6" />
+  <xacro:lrf_gazebo prefix="urg" base_rad="0" rad_range="4.71" min_range="0.10" max_range="5.6" />
   <raspimouse_on_gazebo/>
 </robot>

File: raspimouse_description/urdf/raspimouse.urdf.xacro (robot description, xacro)
@@ -1,66 +1 @@
-<?xml version="1.0"?>
-<robot name="raspimouse_on_gazebo"
-       xmlns:sensor="http://playerstage.sourceforge.net/gazebo/xmlschema/#sensor"
-       xmlns:controller="http://playerstage.sourceforge.net/gazebo/xmlschema/#controller"
-       xmlns:interface="http://playerstage.sourceforge.net/gazebo/xmlschema/#interface"
-       xmlns:xacro="http://ros.org/wiki/xacro">
-  <xacro:include filename="$(find raspimouse_description)/urdf/body/body.urdf.xacro"/>
-  <xacro:include filename="$(find raspimouse_description)/urdf/wheel/wheel.urdf.xacro"/>
-  <xacro:include filename="$(find raspimouse_description)/urdf/sensors/lightsens.urdf.xacro"/>
-  <!-- =============== Link & Joint =============== -->
-  <!-- Base -->
-  <link name="base_footprint"/>
-  <xacro:base parent="base_footprint">
-    <origin xyz="0 0 0.00185"/>
-  </xacro:base>
-  <!-- Wheel -->
-  <xacro:wheel prefix="right" parent="base_link">
-    <origin xyz="0 -0.0425 0.02215" rpy="1.57 0 0"/>
-    <axis xyz="0 0 -1"/>
-  </xacro:wheel>
-  <xacro:wheel prefix="left" parent="base_link">
-    <origin xyz="0 0.0425 0.02215" rpy="-1.57 0 0"/>
-    <axis xyz="0 0 1"/>
-  </xacro:wheel>
-  <!-- Sensors -->
-  <xacro:light_sensor prefix="rf" parent="base_link">
-    <origin xyz="0.04 -0.045 0.032" rpy="0 0 0"/>
-  </xacro:light_sensor>
-  <xacro:light_sensor prefix="rs" parent="base_link">
-    <origin xyz="0.059 -0.01 0.032" rpy="0 0 -1.04"/>
-  </xacro:light_sensor>
-  <xacro:light_sensor prefix="ls" parent="base_link">
-    <origin xyz="0.059 0.01 0.032" rpy="0 0 1.04"/>
-  </xacro:light_sensor>
-  <xacro:light_sensor prefix="lf" parent="base_link">
-    <origin xyz="0.04 0.045 0.032" rpy="0 0 0"/>
-  </xacro:light_sensor>
-  <!-- ===============  Transmission =============== -->
-  <!-- PositionJointInterface: requires position -->
-  <!-- <xacro:wheel_trans prefix="right" interface="PositionJointInterface"/> -->
-  <!-- <xacro:wheel_trans prefix="left" interface="PositionJointInterface"/>  -->
-  <!-- VelocityJointInterface: requires position, velocity -->
-  <!-- for DiffDriveController -->
-  <xacro:wheel_trans prefix="right" interface="VelocityJointInterface"/>
-  <xacro:wheel_trans prefix="left" interface="VelocityJointInterface"/>
-  <!-- EffortJointInterface: requires position, velocity, effort -->
-  <!-- <xacro:wheel_trans prefix="right" interface="EffortJointInterface"/> -->
-  <!-- <xacro:wheel_trans prefix="left" interface="EffortJointInterface"/>  -->
-  <!-- =============== Gazebo =============== -->
-  <gazebo>
-    <plugin name="gazebo_ros_control" filename="libgazebo_ros_control.so">
-      <robotNamespace>raspimouse_on_gazebo</robotNamespace>
-    </plugin>
-  </gazebo>
-  <!-- Base -->
-  <xacro:base_gazebo/>
-  <!-- Wheel -->
-  <xacro:wheel_gazebo prefix="right"/>
-  <xacro:wheel_gazebo prefix="left"/>
-  <!-- Sensors -->
-  <xacro:lightsensor_gazebo prefix="rf" base_rad="0" rad_range="0.3" min_range="0.01" max_range="0.6"/>
-  <xacro:lightsensor_gazebo prefix="rs" base_rad="-1.04" rad_range="0.3" min_range="0.01" max_range="0.6"/>
-  <xacro:lightsensor_gazebo prefix="ls" base_rad="1.04" rad_range="0.3" min_range="0.01" max_range="0.6"/>
-  <xacro:lightsensor_gazebo prefix="lf" base_rad="0" rad_range="0.3" min_range="0.01" max_range="0.6"/>
-  <raspimouse_on_gazebo/>
-</robot>
+../robots/raspimouse.urdf.xacro

File: raspimouse_description/urdf/raspimouse_urg.urdf.xacro (robot description, xacro)
@@ -1,66 +1 @@
-<?xml version="1.0"?>
-<robot name="raspimouse_on_gazebo"
-       xmlns:sensor="http://playerstage.sourceforge.net/gazebo/xmlschema/#sensor"
-       xmlns:controller="http://playerstage.sourceforge.net/gazebo/xmlschema/#controller"
-       xmlns:interface="http://playerstage.sourceforge.net/gazebo/xmlschema/#interface"
-       xmlns:xacro="http://ros.org/wiki/xacro">
-  <xacro:include filename="$(find raspimouse_description)/urdf/body/body_urg.urdf.xacro"/>
-  <xacro:include filename="$(find raspimouse_description)/urdf/wheel/wheel.urdf.xacro"/>
-  <xacro:include filename="$(find raspimouse_description)/urdf/sensors/lightsens.urdf.xacro"/>
-  <xacro:include filename="$(find raspimouse_description)/urdf/sensors/lrf.urdf.xacro"/>
-  <!-- =============== Link & Joint =============== -->
-  <!-- Base -->
-  <link name="base_footprint"/>
-  <xacro:base parent="base_footprint">
-    <origin xyz="0 0 0.00185"/>
-  </xacro:base>
-  <!-- Wheel -->
-  <xacro:wheel prefix="right" parent="base_link">
-    <origin xyz="0 -0.0425 0.02215" rpy="1.57 0 0"/>
-    <axis xyz="0 0 -1"/>
-  </xacro:wheel>
-  <xacro:wheel prefix="left" parent="base_link">
-    <origin xyz="0 0.0425 0.02215" rpy="-1.57 0 0"/>
-    <axis xyz="0 0 1"/>
-  </xacro:wheel>
-  <!-- Sensors -->
-  <xacro:light_sensor prefix="rf" parent="base_link">
-    <origin xyz="0.04 -0.045 0.032" rpy="0 0 0"/>
-  </xacro:light_sensor>
-  <xacro:light_sensor prefix="rs" parent="base_link">
-    <origin xyz="0.059 -0.01 0.032" rpy="0 0 -1.04"/>
-  </xacro:light_sensor>
-  <xacro:light_sensor prefix="ls" parent="base_link">
-    <origin xyz="0.059 0.01 0.032" rpy="0 0 1.04"/>
-  </xacro:light_sensor>
-  <xacro:light_sensor prefix="lf" parent="base_link">
-    <origin xyz="0.04 0.045 0.032" rpy="0 0 0"/>
-  </xacro:light_sensor>
-  <xacro:lrf_sensor prefix="urg_lrf_link" parent="base_link">
-    <origin xyz="0.0 0.0 0.14060" rpy="0 0 0"/>
-    <!-- <origin xyz="0.0 0.0 0.18745" rpy="0 0 0"/> -->
-  </xacro:lrf_sensor>
-  <!-- ===============  Transmission =============== -->
-  <!-- <xacro:wheel_trans prefix="right" interface="EffortJointInterface"/> -->
-  <!-- <xacro:wheel_trans prefix="left" interface="EffortJointInterface"/> -->
-  <xacro:wheel_trans prefix="right" interface="VelocityJointInterface"/>
-  <xacro:wheel_trans prefix="left" interface="VelocityJointInterface"/>
-  <!-- =============== Gazebo =============== -->
-  <gazebo>
-    <plugin name="gazebo_ros_control" filename="libgazebo_ros_control.so">
-      <robotNamespace>raspimouse_on_gazebo</robotNamespace>
-    </plugin>
-  </gazebo>
-  <!-- Base -->
-  <xacro:base_gazebo/>
-  <!-- Wheel -->
-  <xacro:wheel_gazebo prefix="right"/>
-  <xacro:wheel_gazebo prefix="left"/>
-  <!-- Sensors -->
-  <xacro:lightsensor_gazebo prefix="rf" base_rad="0" rad_range="0.3" min_range="0.01" max_range="0.6"/>
-  <xacro:lightsensor_gazebo prefix="rs" base_rad="-1.04" rad_range="0.3" min_range="0.01" max_range="0.6"/>
-  <xacro:lightsensor_gazebo prefix="ls" base_rad="1.04" rad_range="0.3" min_range="0.01" max_range="0.6"/>
-  <xacro:lightsensor_gazebo prefix="lf" base_rad="0" rad_range="0.3" min_range="0.01" max_range="0.6"/>
-  <xacro:lrf_gazebo prefix="urg" base_rad="0" rad_range="4.71" min_range="0.10" max_range="5.6"/>
-  <raspimouse_on_gazebo/>
-</robot>
+../robots/raspimouse_urg.urdf.xacro
